File: rgb_oled_0.95in.kicad_pcb (KiCad board)
At the start: 2 copper layers, 39 x 25 mm, 14 parts, among them J1 PMOD, U1 LMR62014, U2 UG-9664HDDAG01

Commit message: Add nicer silk
Parts:
- R3: value 500K -> 510K
Changed lines of the file:
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@@
       (effects (font (size 1 1) (thickness 0.15)) (justify mirror))
     )
-    (fp_text value 500K (at 0 -1.43 270) (layer B.Fab)
+    (fp_text value 510K (at 0 -1.43 270) (layer B.Fab)
       (effects (font (size 1 1) (thickness 0.15)) (justify mirror))
     )
